Commit message: Replace sensor kit template with multi-sensor sample

File: skku_sensor_kit_description/urdf/sensor_kit.xacro (robot description, xacro)
@@ -3,7 +3,9 @@
   <xacro:macro name="sensor_kit_macro" params="parent x y z roll pitch yaw">
     <xacro:include filename="$(find velodyne_description)/urdf/VLP-16.urdf.xacro"/>
-    <xacro:include filename="$(find autoware_sample_sensor_kit_description)/sensor/vls/urdf/VLS-128.urdf.xacro"/>
+    <xacro:include filename="$(find skku_sensor_kit_description)/sensor/vls/urdf/VLS-128.urdf.xacro"/>
+    <xacro:include filename="$(find skku_sensor_kit_description)/sensor/camera/urdf/monocular_camera.xacro"/>
+    <xacro:include filename="$(find skku_sensor_kit_description)/sensor/imu/urdf/imu.xacro"/>
     <xacro:arg name="gpu" default="false"/>
-    <xacro:arg name="config_dir" default="$(find autoware_sample_sensor_kit_description)/config"/>
+    <xacro:arg name="config_dir" default="$(find skku_sensor_kit_description)/config"/>
     <xacro:property name="sensor_kit_base_link" default="sensor_kit_base_link"/>
     <joint name="${sensor_kit_base_link}_joint" type="fixed">
@@ -28,4 +30,171 @@
       />
     </xacro:VLS-128>
+    <xacro:VLP-16 parent="sensor_kit_base_link" name="velodyne_left" topic="/points_raw" hz="10" samples="220" gpu="$(arg gpu)">
+      <origin
+        xyz="${calibration['sensor_kit_base_link']['velodyne_left_base_link']['x']}
+             ${calibration['sensor_kit_base_link']['velodyne_left_base_link']['y']}
+             ${calibration['sensor_kit_base_link']['velodyne_left_base_link']['z']}"
+        rpy="${calibration['sensor_kit_base_link']['velodyne_left_base_link']['roll']}
+             ${calibration['sensor_kit_base_link']['velodyne_left_base_link']['pitch']}
+             ${calibration['sensor_kit_base_link']['velodyne_left_base_link']['yaw']}"
+      />
+    </xacro:VLP-16>
+    <xacro:VLP-16 parent="sensor_kit_base_link" name="velodyne_right" topic="/points_raw" hz="10" samples="220" gpu="$(arg gpu)">
+      <origin
+        xyz="${calibration['sensor_kit_base_link']['velodyne_right_base_link']['x']}
+             ${calibration['sensor_kit_base_link']['velodyne_right_base_link']['y']}
+             ${calibration['sensor_kit_base_link']['velodyne_right_base_link']['z']}"
+        rpy="${calibration['sensor_kit_base_link']['velodyne_right_base_link']['roll']}
+             ${calibration['sensor_kit_base_link']['velodyne_right_base_link']['pitch']}
+             ${calibration['sensor_kit_base_link']['velodyne_right_base_link']['yaw']}"
+      />
+    </xacro:VLP-16>
+    <!-- camera -->
+    <xacro:monocular_camera_macro
+      name="traffic_light_right_camera/camera"
+      parent="sensor_kit_base_link"
+      namespace=""
+      x="${calibration['sensor_kit_base_link']['traffic_light_right_camera/camera_link']['x']}"
+      y="${calibration['sensor_kit_base_link']['traffic_light_right_camera/camera_link']['y']}"
+      z="${calibration['sensor_kit_base_link']['traffic_light_right_camera/camera_link']['z']}"
+      roll="${calibration['sensor_kit_base_link']['traffic_light_right_camera/camera_link']['roll']}"
+      pitch="${calibration['sensor_kit_base_link']['traffic_light_right_camera/camera_link']['pitch']}"
+      yaw="${calibration['sensor_kit_base_link']['traffic_light_right_camera/camera_link']['yaw']}"
+      fps="30"
+      width="800"
+      height="400"
+      fov="1.3"
+    />
+    <xacro:monocular_camera_macro
+      name="traffic_light_left_camera/camera"
+      parent="sensor_kit_base_link"
+      namespace=""
+      x="${calibration['sensor_kit_base_link']['traffic_light_left_camera/camera_link']['x']}"
+      y="${calibration['sensor_kit_base_link']['traffic_light_left_camera/camera_link']['y']}"
+      z="${calibration['sensor_kit_base_link']['traffic_light_left_camera/camera_link']['z']}"
+      roll="${calibration['sensor_kit_base_link']['traffic_light_left_camera/camera_link']['roll']}"
+      pitch="${calibration['sensor_kit_base_link']['traffic_light_left_camera/camera_link']['pitch']}"
+      yaw="${calibration['sensor_kit_base_link']['traffic_light_left_camera/camera_link']['yaw']}"
+      fps="30"
+      width="800"
+      height="400"
+      fov="1.3"
+    />
+    <xacro:monocular_camera_macro
+      name="camera0/camera"
+      parent="sensor_kit_base_link"
+      namespace=""
+      x="${calibration['sensor_kit_base_link']['camera0/camera_link']['x']}"
+      y="${calibration['sensor_kit_base_link']['camera0/camera_link']['y']}"
+      z="${calibration['sensor_kit_base_link']['camera0/camera_link']['z']}"
+      roll="${calibration['sensor_kit_base_link']['camera0/camera_link']['roll']}"
+      pitch="${calibration['sensor_kit_base_link']['camera0/camera_link']['pitch']}"
+      yaw="${calibration['sensor_kit_base_link']['camera0/camera_link']['yaw']}"
+      fps="30"
+      width="800"
+      height="400"
+      fov="1.3"
+    />
+    <xacro:monocular_camera_macro
+      name="camera1/camera"
+      parent="sensor_kit_base_link"
+      namespace=""
+      x="${calibration['sensor_kit_base_link']['camera1/camera_link']['x']}"
+      y="${calibration['sensor_kit_base_link']['camera1/camera_link']['y']}"
+      z="${calibration['sensor_kit_base_link']['camera1/camera_link']['z']}"
+      roll="${calibration['sensor_kit_base_link']['camera1/camera_link']['roll']}"
+      pitch="${calibration['sensor_kit_base_link']['camera1/camera_link']['pitch']}"
+      yaw="${calibration['sensor_kit_base_link']['camera1/camera_link']['yaw']}"
+      fps="30"
+      width="800"
+      height="400"
+      fov="1.3"
+    />
+    <xacro:monocular_camera_macro
+      name="camera2/camera"
+      parent="sensor_kit_base_link"
+      namespace=""
+      x="${calibration['sensor_kit_base_link']['camera2/camera_link']['x']}"
+      y="${calibration['sensor_kit_base_link']['camera2/camera_link']['y']}"
+      z="${calibration['sensor_kit_base_link']['camera2/camera_link']['z']}"
+      roll="${calibration['sensor_kit_base_link']['camera2/camera_link']['roll']}"
+      pitch="${calibration['sensor_kit_base_link']['camera2/camera_link']['pitch']}"
+      yaw="${calibration['sensor_kit_base_link']['camera2/camera_link']['yaw']}"
+      fps="30"
+      width="800"
+      height="400"
+      fov="1.3"
+    />
+    <xacro:monocular_camera_macro
+      name="camera3/camera"
+      parent="sensor_kit_base_link"
+      namespace=""
+      x="${calibration['sensor_kit_base_link']['camera3/camera_link']['x']}"
+      y="${calibration['sensor_kit_base_link']['camera3/camera_link']['y']}"
+      z="${calibration['sensor_kit_base_link']['camera3/camera_link']['z']}"
+      roll="${calibration['sensor_kit_base_link']['camera3/camera_link']['roll']}"
+      pitch="${calibration['sensor_kit_base_link']['camera3/camera_link']['pitch']}"
+      yaw="${calibration['sensor_kit_base_link']['camera3/camera_link']['yaw']}"
+      fps="30"
+      width="800"
+      height="400"
+      fov="1.3"
+    />
+    <xacro:monocular_camera_macro
+      name="camera4/camera"
+      parent="sensor_kit_base_link"
+      namespace=""
+      x="${calibration['sensor_kit_base_link']['camera4/camera_link']['x']}"
+      y="${calibration['sensor_kit_base_link']['camera4/camera_link']['y']}"
+      z="${calibration['sensor_kit_base_link']['camera4/camera_link']['z']}"
+      roll="${calibration['sensor_kit_base_link']['camera4/camera_link']['roll']}"
+      pitch="${calibration['sensor_kit_base_link']['camera4/camera_link']['pitch']}"
+      yaw="${calibration['sensor_kit_base_link']['camera4/camera_link']['yaw']}"
+      fps="30"
+      width="800"
+      height="400"
+      fov="1.3"
+    />
+    <xacro:monocular_camera_macro
+      name="camera5/camera"
+      parent="sensor_kit_base_link"
+      namespace=""
+      x="${calibration['sensor_kit_base_link']['camera5/camera_link']['x']}"
+      y="${calibration['sensor_kit_base_link']['camera5/camera_link']['y']}"
+      z="${calibration['sensor_kit_base_link']['camera5/camera_link']['z']}"
+      roll="${calibration['sensor_kit_base_link']['camera5/camera_link']['roll']}"
+      pitch="${calibration['sensor_kit_base_link']['camera5/camera_link']['pitch']}"
+      yaw="${calibration['sensor_kit_base_link']['camera5/camera_link']['yaw']}"
+      fps="30"
+      width="800"
+      height="400"
+      fov="1.3"
+    />
+    <!-- gnss -->
+    <xacro:imu_macro
+      name="gnss"
+      parent="sensor_kit_base_link"
+      namespace=""
+      x="${calibration['sensor_kit_base_link']['gnss_link']['x']}"
+      y="${calibration['sensor_kit_base_link']['gnss_link']['y']}"
+      z="${calibration['sensor_kit_base_link']['gnss_link']['z']}"
+      roll="${calibration['sensor_kit_base_link']['gnss_link']['roll']}"
+      pitch="${calibration['sensor_kit_base_link']['gnss_link']['pitch']}"
+      yaw="${calibration['sensor_kit_base_link']['gnss_link']['yaw']}"
+      fps="100"
+    />
+    <!-- imu -->
+    <xacro:imu_macro
+      name="tamagawa/imu"
+      parent="sensor_kit_base_link"
+      namespace=""
+      x="${calibration['sensor_kit_base_link']['tamagawa/imu_link']['x']}"
+      y="${calibration['sensor_kit_base_link']['tamagawa/imu_link']['y']}"
+      z="${calibration['sensor_kit_base_link']['tamagawa/imu_link']['z']}"
+      roll="${calibration['sensor_kit_base_link']['tamagawa/imu_link']['roll']}"
+      pitch="${calibration['sensor_kit_base_link']['tamagawa/imu_link']['pitch']}"
+      yaw="${calibration['sensor_kit_base_link']['tamagawa/imu_link']['yaw']}"
+      fps="100"
+    />
   </xacro:macro>
 </robot>

File: skku_sensor_kit_description/urdf/sensors.xacro (robot description, xacro)
@@ -14,3 +14,15 @@
     yaw="${calibration['base_link']['sensor_kit_base_link']['yaw']}"
   />
+  <!-- embedded sensors -->
+  <xacro:include filename="$(find velodyne_description)/urdf/VLP-16.urdf.xacro"/>
+  <xacro:VLP-16 parent="base_link" name="velodyne_rear" topic="velodyne_rear/velodyne_points" hz="10" samples="220" gpu="false">
+    <origin
+      xyz="${calibration['base_link']['velodyne_rear_base_link']['x']}
+           ${calibration['base_link']['velodyne_rear_base_link']['y']}
+           ${calibration['base_link']['velodyne_rear_base_link']['z']}"
+      rpy="${calibration['base_link']['velodyne_rear_base_link']['roll']}
+           ${calibration['base_link']['velodyne_rear_base_link']['pitch']}
+           ${calibration['base_link']['velodyne_rear_base_link']['yaw']}"
+    />
+  </xacro:VLP-16>
 </robot>
